File: ClassicRev4.kicad_pcb (KiCad board)
At the start: 2 copper layers, 65 x 50 mm, 64 parts, among them IC1 7805TV, IC2 MEGA8-P, IC3 74141N, Q1 IRF740, Q2 16MHz, Q3 2N7000, Q4 2N7000, Q5 2N7000, Q6 2N7000

Commit message: Initial commit Classic Rev4c
Parts:
- added TP4: HVD, Recovered:TESTPAD_P1-13, F.Cu at (120.9, 131.1)
- C2, C5, C6, C7, C8: footprint NixieClockModule:rcl-C050-024X044 -> NixieClockMaster:C025-024X044
- D1, D2: footprint Diodes_ThroughHole:Diode_DO-41_SOD81_Horizontal_RM10 -> NixieClockMaster:Diode_DO-41_1N4001
- IC3: value 74141N -> K155ID1
- Q1: footprint NixieClockModule:TRANSISTOR-POWER_TO220BV -> NixieClockMaster:TRANSISTOR-POWER_TO220BV
- SV1, SV4, SV6: footprint NixieClockModule:Header_MA04-1 -> NixieClockMaster:Header_MA04-1
- SV2: footprint NixieClockModule:Header_MA04-1 -> NixieClockMaster:Header_MA06-1
- SV3: footprint NixieClockModule:Header_MA06-1 -> NixieClockMaster:Header_MA06-1
- moved TP3 67.5 mm to (180.2, 131.3)
- moved R7 26.1 mm to (141.1, 115.5), turned to 90 degrees
- moved TP2 5.48 mm to (177.7, 127.5)
- moved C2 1.81 mm to (141.0, 110.9)
- moved C8 1.03 mm to (161.8, 94.8)
- moved C5 1.00 mm to (161.8, 92.4)
- moved C6 1.00 mm to (144.9, 92.3)
- moved C7 0.99 mm to (144.9, 94.8)
- moved SV2 0.72 mm to (131.7, 92.8)
- moved TP1 0.50 mm to (180.2, 127.5)
- renumbered REF** to MH1, REF** to MH2, REF** to MH3, REF** to MH4
Connections:
- net /N$1 renamed /TICK_BASE
- net /N$31 renamed /B_GATE
- net /N$32 renamed /R_GATE
- net /N$35 renamed /G_GATE
- IC3 pad 1: /CATHODE_8 -> /CATHODE_9
- IC3 pad 2: /CATHODE_9 -> /CATHODE_8
- SV2 pad 1: GND -> /VCC
- SV2 pad 2: /DLS -> /ANODE5
- SV2 pad 4: /VCC -> /DLS
- SV5 pad 10: /CATHODE_8 -> /CATHODE_9
- SV5 pad 9: /CATHODE_9 -> /CATHODE_8
Routing:
- net /ANODE5: track 11.8 -> 56.9 mm, vias 0 -> 2
- net /ANODE6: track 18.0 -> 61.6 mm, vias 0 -> 1
- net /VCC: track 188.6 -> 211.9 mm
- net GND: track 328.4 -> 341.0 mm, vias 0 -> 1
- net /VIN: track 31.5 -> 34.9 mm
- net /BTN1: track 15.0 -> 18.0 mm
- net /DRAIN: track 26.8 -> 23.8 mm
- net /CATHODE_0: track 14.9 -> 12.2 mm
- net /DLS: track 45.9 -> 48.4 mm
- net Net-(R6-Pad1): track 4.66 -> 3.13 mm
- net /170V: track 121.1 -> 122.5 mm
- net /HVD: track 44.3 -> 45.4 mm
- net /DIGIT_A: track 61.0 -> 60.0 mm
- net /DIGIT_D: track 62.1 -> 61.3 mm
- net /DIGIT_C: track 39.8 -> 39.0 mm
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Other:
- net class HighPower added: clearance 0.254, trace_width 0.4, via_dia 0.6, via_drill 0.4
- board text added: "20180906"
- board text added: "Rev4c"
- board text removed: "20160927"
- board text removed: "Rev4b"

Commit message: KiCad 5
Parts:
- moved SV1 12.0 mm to (118.8, 112.3)
- moved IC1 11.9 mm to (116.2, 101.1)
- moved R11 11.7 mm to (139.2, 94.5), turned to 0 degrees
- moved R8 5.44 mm to (124.9, 103.2), turned to 0 degrees
- moved LED1 3.78 mm to (129.9, 104.5), turned to 0 degrees
- moved C9 2.39 mm to (125.9, 98.6), turned to 90 degrees
- moved SV2 2.35 mm to (132.8, 90.7)
- moved Q1 2.03 mm to (116.3, 124.4)
- moved IC3 2.00 mm to (134.1, 130.8)
- moved R15 2.00 mm to (151.5, 134.0)
- moved R16 2.00 mm to (154.1, 134.0)
- moved R17 2.00 mm to (156.6, 134.0)
- moved R19 2.00 mm to (176.3, 133.9)
- moved R20 2.00 mm to (173.8, 133.9)
- moved R21 2.00 mm to (171.2, 133.9)
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Routing:
- net GND: track 341.0 -> 312.7 mm, vias 1 -> 2
- net /VCC: track 211.9 -> 198.5 mm
- net /VIN: track 34.9 -> 47.6 mm
- net /DLS: track 48.4 -> 41.7 mm
- net /DIGIT_A: track 60.0 -> 64.0 mm
- net /DIGIT_D: track 61.3 -> 65.0 mm
- net /170V: track 122.5 -> 125.6 mm, vias 1 -> 2
- net /ANODE6: track 61.6 -> 63.7 mm
- net /DRAIN: track 23.8 -> 25.9 mm
- net Net-(Q5-Pad1): track 22.1 -> 24.1 mm
- net /SCL: track 14.3 -> 16.3 mm
- net /SDA: track 13.6 -> 15.6 mm
- net Net-(Q4-Pad1): track 28.2 -> 30.2 mm
- net Net-(OK6-Pad3): track 8.15 -> 10.1 mm
- net Net-(OK5-Pad3): track 9.94 -> 11.9 mm
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Other:
- board size 65 x 50 mm -> 69 x 54 mm

Commit message: Add copyright and license notices
Routing:
- added copper zone on B.Cu, net GND
Other:
- board text added: "Copyright 2019 Ian Sparkes https://www.nixieclock.biz"
- board text added: "License CC-BY-SA"
Changed lines of the file:
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@@
   (general
     (thickness 1.6)
-    (drawings 6)
+    (drawings 10)
     (tracks 701)
     (zones 0)
@@
       (net 1 GND))
   )
+  (gr_text "License CC-BY-SA" (at 164.60372 127.3292) (layer B.SilkS)
+    (effects (font (size 1 1) (thickness 0.2)) (justify mirror))
+  )
+  (gr_text "Copyright 2019 Ian Sparkes\nhttps://www.nixieclock.biz" (at 132.95372 123.1492) (layer B.SilkS)
+    (effects (font (size 0.75 0.75) (thickness 0.1)) (justify mirror))
+  )
+  (gr_text "License CC-BY-SA" (at 164.69372 126.9692) (layer F.SilkS)
+    (effects (font (size 1 1) (thickness 0.2)))
+  )
+  (gr_text "Copyright 2019 Ian Sparkes\nhttps://www.nixieclock.biz" (at 132.95372 123.3192) (layer F.SilkS)
+    (effects (font (size 0.75 0.75) (thickness 0.1)))
+  )
   (gr_text 20180906 (at 137.85342 131.4511) (layer F.SilkS)
     (effects (font (size 0.75 0.75) (thickness 0.1)))
@@
   (segment (start 150.58593 109.99902) (end 152.49093 111.90402) (width 0.254) (layer B.Cu) (net 68) (status 20))
   (segment (start 147.72843 109.99902) (end 150.58593 109.99902) (width 0.254) (layer B.Cu) (net 68) (status 10))
+  (zone (net 1) (net_name GND) (layer B.Cu) (hatch edge 0.508)
+    (connect_pads (clearance 0.508))
+    (min_thickness 0.254)
+    (fill yes (arc_segments 16) (thermal_gap 0.508) (thermal_bridge_width 0.508))
+    (polygon
+      (pts
+        (xy 115.86372 87.6792) (xy 184.86372 87.6892) (xy 184.87372 141.6792) (xy 115.86372 141.6792)
+      )
+    )
+  )
 )
